File: fastlinefollower_l298n.kicad_pcb (KiCad board)
At the start: 2 copper layers, 88 x 68 mm, 24 parts, among them J1 IR_conn, J2 Motor1, J3 Motor2, Q1 BC547, Q2 BC547, SW1 Run, SW2 Calibrate, U1 L298N, U2 LM7805_TO220

Commit message: updates260523
Parts:
- moved Q1 101.7 mm to (150.7, 130.0)
- moved SW1 91.6 mm to (116.8, 98.8)
- moved SW2 87.4 mm to (123.2, 95.2), turned to 180 degrees
- moved Q2 82.6 mm to (167.0, 105.7), turned to -90 degrees
- moved D6 55.6 mm to (124.4, 125.3), turned to 90 degrees
- moved D3 45.6 mm to (179.6, 115.2)
- moved D4 45.6 mm to (173.6, 115.2)
- moved D7 45.6 mm to (183.6, 125.3)
- moved D8 45.6 mm to (169.6, 125.3)
- moved D1 41.9 mm to (134.4, 115.2), turned to -90 degrees
- moved D5 27.6 mm to (138.4, 125.3), turned to 90 degrees
- moved C4 27.4 mm to (141.5, 114.8), turned to 90 degrees
- moved C3 23.7 mm to (166.5, 129.2)
- moved U1 21.3 mm to (145.1, 125.3), turned to 0 degrees
- moved C2 17.0 mm to (131.0, 75.0), turned to 0 degrees
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Connections:
- A1 pad 8: /PWM_1 -> /PWM_2
- A1 pad 9: /PWM_2 -> /PWM_1
Routing:
- net +5V: track 0.00 -> 74.2 mm
- net VS: track 0.00 -> 66.3 mm
- net /PWM_2: track 0.00 -> 62.6 mm, vias 0 -> 2
- net Net-(Q1-B): track 0.00 -> 62.1 mm, vias 0 -> 4
- net /M1_B: track 0.00 -> 33.6 mm, vias 0 -> 2
- net /M2_A: track 0.00 -> 32.3 mm, vias 0 -> 2
- net /PWM_1: track 0.00 -> 25.7 mm
- net /M2_B: track 0.00 -> 20.1 mm, vias 0 -> 2
- net /IN4: track 0.00 -> 18.4 mm
- net /M1_A: track 0.00 -> 14.8 mm
- net Net-(Q2-B): track 0.00 -> 12.3 mm
- net /DIR_2: track 0.00 -> 7.39 mm
- net /DIR_1: track 0.00 -> 7.39 mm
- net /IR8: track 0.00 -> 6.37 mm
- net /IR7: track 0.00 -> 6.37 mm
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- added copper zone on B.Cu, net GND
