File: fastlinefollower_l298n.kicad_sch (KiCad schematic)
At the start: 24 parts, among them J1 IR_conn, J2 Motor1, J3 Motor2, Q1 BC547, Q2 BC547, SW1 Run, SW2 Calibrate, U1 L298N, U2 LM7805_TO220

Commit message: updates260523
Connections:
- net PWM_1: now also A1.9 (D6); no longer A1.8 (D5)
- net PWM_2: now also A1.8 (D5); no longer A1.9 (D6)
Changed lines of the file:
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@@
     (effects (font (size 1.27 1.27)) (justify left bottom))
   )
-  (label "PWM_2" (at 106.68 64.77 0) (fields_autoplaced)
+  (label "PWM_1" (at 106.68 64.77 0) (fields_autoplaced)
     (effects (font (size 1.27 1.27)) (justify left bottom))
   )
@@
     (effects (font (size 1.27 1.27)) (justify left bottom))
   )
-  (label "PWM_1" (at 106.68 62.23 0) (fields_autoplaced)
+  (label "PWM_2" (at 106.68 62.23 0) (fields_autoplaced)
     (effects (font (size 1.27 1.27)) (justify left bottom))
   )
@@
     (pin "1")
     (instances
-      (project "fastlinefollower"
+      (project "fastlinefollower_l298n"
         (path "/12d22a33-b5ed-48ef-8dcf-cecf4d5020b2"
           (reference "#PWR012") (unit 1)
@@
     (pin "9")
     (instances
-      (project "fastlinefollower"
+      (project "fastlinefollower_l298n"
         (path "/12d22a33-b5ed-48ef-8dcf-cecf4d5020b2"
           (reference "A1") (unit 1)
@@
     (pin "2")
     (instances
-      (project "fastlinefollower"
+      (project "fastlinefollower_l298n"
         (path "/12d22a33-b5ed-48ef-8dcf-cecf4d5020b2"
           (reference "D2") (unit 1)
@@
     (pin "1")
     (instances
-      (project "fastlinefollower"
+      (project "fastlinefollower_l298n"
         (path "/12d22a33-b5ed-48ef-8dcf-cecf4d5020b2"
           (reference "#PWR014") (unit 1)
@@
     (pin "2")
     (instances
-      (project "fastlinefollower"
+      (project "fastlinefollower_l298n"
         (path "/12d22a33-b5ed-48ef-8dcf-cecf4d5020b2"
           (reference "R2") (unit 1)
@@
     (pin "2")
     (instances
-      (project "fastlinefollower"
+      (project "fastlinefollower_l298n"
         (path "/12d22a33-b5ed-48ef-8dcf-cecf4d5020b2"
           (reference "D6") (unit 1)
@@
     (pin "3")
     (instances
-      (project "fastlinefollower"
+      (project "fastlinefollower_l298n"
         (path "/12d22a33-b5ed-48ef-8dcf-cecf4d5020b2"
           (reference "U2") (unit 1)
@@
     (pin "1")
     (instances
-      (project "fastlinefollower"
+      (project "fastlinefollower_l298n"
         (path "/12d22a33-b5ed-48ef-8dcf-cecf4d5020b2"
           (reference "#PWR011") (unit 1)
@@
     (pin "2")
     (instances
-      (project "fastlinefollower"
+      (project "fastlinefollower_l298n"
         (path "/12d22a33-b5ed-48ef-8dcf-cecf4d5020b2"
           (reference "D3") (unit 1)
@@
     (pin "2")
     (instances
-      (project "fastlinefollower"
+      (project "fastlinefollower_l298n"
         (path "/12d22a33-b5ed-48ef-8dcf-cecf4d5020b2"
           (reference "D7") (unit 1)
@@
     (pin "2")
     (instances
-      (project "fastlinefollower"
+      (project "fastlinefollower_l298n"
         (path "/12d22a33-b5ed-48ef-8dcf-cecf4d5020b2"
           (reference "C4") (unit 1)
@@
     (pin "2")
     (instances
-      (project "fastlinefollower"
+      (project "fastlinefollower_l298n"
         (path "/12d22a33-b5ed-48ef-8dcf-cecf4d5020b2"
           (reference "J2") (unit 1)
@@
     (pin "2")
     (instances
-      (project "fastlinefollower"
+      (project "fastlinefollower_l298n"
         (path "/12d22a33-b5ed-48ef-8dcf-cecf4d5020b2"
           (reference "D4") (unit 1)
@@
     (pin "9")
     (instances
-      (project "fastlinefollower"
+      (project "fastlinefollower_l298n"
         (path "/12d22a33-b5ed-48ef-8dcf-cecf4d5020b2"
           (reference "U1") (unit 1)
@@
     (pin "2")
     (instances
-      (project "fastlinefollower"
+      (project "fastlinefollower_l298n"
         (path "/12d22a33-b5ed-48ef-8dcf-cecf4d5020b2"
           (reference "D1") (unit 1)
@@
     (pin "2")
     (instances
-      (project "fastlinefollower"
+      (project "fastlinefollower_l298n"
         (path "/12d22a33-b5ed-48ef-8dcf-cecf4d5020b2"
           (reference "SW1") (unit 1)
@@
     (pin "2")
     (instances
-      (project "fastlinefollower"
+      (project "fastlinefollower_l298n"
         (path "/12d22a33-b5ed-48ef-8dcf-cecf4d5020b2"
           (reference "SW2") (unit 1)
@@
     (pin "1")
     (instances
-      (project "fastlinefollower"
+      (project "fastlinefollower_l298n"
         (path "/12d22a33-b5ed-48ef-8dcf-cecf4d5020b2"
           (reference "#PWR010") (unit 1)
@@
     (pin "1")
     (instances
-      (project "fastlinefollower"
+      (project "fastlinefollower_l298n"
         (path "/12d22a33-b5ed-48ef-8dcf-cecf4d5020b2"
           (reference "#PWR08") (unit 1)
@@
     (pin "1")
     (instances
-      (project "fastlinefollower"
+      (project "fastlinefollower_l298n"
         (path "/12d22a33-b5ed-48ef-8dcf-cecf4d5020b2"
           (reference "#PWR09") (unit 1)
@@
     (pin "1")
     (instances
-      (project "fastlinefollower"
+      (project "fastlinefollower_l298n"
         (path "/12d22a33-b5ed-48ef-8dcf-cecf4d5020b2"
           (reference "#PWR015") (unit 1)
@@
     (pin "1")
     (instances
-      (project "fastlinefollower"
+      (project "fastlinefollower_l298n"
         (path "/12d22a33-b5ed-48ef-8dcf-cecf4d5020b2"
           (reference "#PWR02") (unit 1)
@@
     (pin "2")
     (instances
-      (project "fastlinefollower"
+      (project "fastlinefollower_l298n"
         (path "/12d22a33-b5ed-48ef-8dcf-cecf4d5020b2"
           (reference "R1") (unit 1)
@@
     (pin "1")
     (instances
-      (project "fastlinefollower"
+      (project "fastlinefollower_l298n"
         (path "/12d22a33-b5ed-48ef-8dcf-cecf4d5020b2"
           (reference "#PWR01") (unit 1)
@@
     (pin "1")
     (instances
-      (project "fastlinefollower"
+      (project "fastlinefollower_l298n"
         (path "/12d22a33-b5ed-48ef-8dcf-cecf4d5020b2"
           (reference "#PWR06") (unit 1)
@@
     (pin "3")
     (instances
-      (project "fastlinefollower"
+      (project "fastlinefollower_l298n"
         (path "/12d22a33-b5ed-48ef-8dcf-cecf4d5020b2"
           (reference "Q2") (unit 1)
@@
     (pin "1")
     (instances
-      (project "fastlinefollower"
+      (project "fastlinefollower_l298n"
         (path "/12d22a33-b5ed-48ef-8dcf-cecf4d5020b2"
           (reference "#PWR018") (unit 1)
@@
     (pin "2")
     (instances
-      (project "fastlinefollower"
+      (project "fastlinefollower_l298n"
         (path "/12d22a33-b5ed-48ef-8dcf-cecf4d5020b2"
           (reference "D5") (unit 1)
@@
     (pin "2")
     (instances
-      (project "fastlinefollower"
+      (project "fastlinefollower_l298n"
         (path "/12d22a33-b5ed-48ef-8dcf-cecf4d5020b2"
           (reference "C1") (unit 1)
@@
     (pin "2")
     (instances
-      (project "fastlinefollower"
+      (project "fastlinefollower_l298n"
         (path "/12d22a33-b5ed-48ef-8dcf-cecf4d5020b2"
           (reference "C2") (unit 1)
@@
     (pin "9")
     (instances
-      (project "fastlinefollower"
+      (project "fastlinefollower_l298n"
         (path "/12d22a33-b5ed-48ef-8dcf-cecf4d5020b2"
           (reference "J1") (unit 1)
@@
     (pin "2")
     (instances
-      (project "fastlinefollower"
+      (project "fastlinefollower_l298n"
         (path "/12d22a33-b5ed-48ef-8dcf-cecf4d5020b2"
           (reference "J3") (unit 1)
@@
     (pin "1")
     (instances
-      (project "fastlinefollower"
+      (project "fastlinefollower_l298n"
         (path "/12d22a33-b5ed-48ef-8dcf-cecf4d5020b2"
           (reference "#PWR05") (unit 1)
@@
     (pin "1")
     (instances
-      (project "fastlinefollower"
+      (project "fastlinefollower_l298n"
         (path "/12d22a33-b5ed-48ef-8dcf-cecf4d5020b2"
           (reference "#PWR017") (unit 1)
@@
     (pin "1")
     (instances
-      (project "fastlinefollower"
+      (project "fastlinefollower_l298n"
         (path "/12d22a33-b5ed-48ef-8dcf-cecf4d5020b2"
           (reference "#PWR016") (unit 1)
@@
     (pin "2")
     (instances
-      (project "fastlinefollower"
+      (project "fastlinefollower_l298n"
         (path "/12d22a33-b5ed-48ef-8dcf-cecf4d5020b2"
           (reference "D8") (unit 1)
@@
     (pin "1")
     (instances
-      (project "fastlinefollower"
+      (project "fastlinefollower_l298n"
         (path "/12d22a33-b5ed-48ef-8dcf-cecf4d5020b2"
           (reference "#PWR04") (unit 1)
@@
     (pin "1")
     (instances
-      (project "fastlinefollower"
+      (project "fastlinefollower_l298n"
         (path "/12d22a33-b5ed-48ef-8dcf-cecf4d5020b2"
           (reference "#PWR03") (unit 1)
@@
     (pin "1")
     (instances
-      (project "fastlinefollower"
+      (project "fastlinefollower_l298n"
         (path "/12d22a33-b5ed-48ef-8dcf-cecf4d5020b2"
           (reference "#PWR013") (unit 1)
@@
     (pin "1")
     (instances
-      (project "fastlinefollower"
+      (project "fastlinefollower_l298n"
         (path "/12d22a33-b5ed-48ef-8dcf-cecf4d5020b2"
           (reference "#PWR020") (unit 1)
@@
     (pin "2")
     (instances
-      (project "fastlinefollower"
+      (project "fastlinefollower_l298n"
         (path "/12d22a33-b5ed-48ef-8dcf-cecf4d5020b2"
           (reference "C3") (unit 1)
@@
     (pin "3")
     (instances
-      (project "fastlinefollower"
+      (project "fastlinefollower_l298n"
         (path "/12d22a33-b5ed-48ef-8dcf-cecf4d5020b2"
           (reference "Q1") (unit 1)
