File: fastlinefollower_tbfng.kicad_sch (KiCad schematic)
At the start: 14 parts, among them J1 IR_conn, J2 Motor1, J3 Motor2, Q1 BC547, Q2 BC547, SW1 Run, SW2 Calibrate, U1 TB6612FNG_Module, U2 LM7805_TO220

Commit message: basic layout done
Parts:
- removed Q1, Q2: BC547, Package_TO_SOT_THT:TO-92_Inline, symbol Transistor_BJT:BC547
- removed R1, R2: R, Resistor_THT:R_Axial_DIN0207_L6.3mm_D2.5mm_P10.16mm_Horizontal, symbol Device:R
- U1: footprint (none) -> sche:TB1266FNG_Module
Connections:
- net DIR_1 is gone; now on net AIN2: A1.10 (D7)
- net DIR_2 is gone; now on net BIN1: A1.11 (D8)
- net +5V: now also U1.2 (Vcc)
- net GND: now also U1.16 (GND), U1.3 (GND), U1.8 (GND)
- net M1_A: now also U1.4 (A1_Out)
- net M1_B: now also U1.5 (A2_Out)
- net M2_A: now also U1.6 (B1_Out)
- net M2_B: now also U1.7 (B2_Out)
- net PWM_1: now also U1.9 (PWM_A)
- net PWM_2: now also A1.13 (D10), U1.15 (PWM_B); no longer A1.9 (D6)
- net VS: now also U1.1 (VM)
- net BIN2: now reaches A1.12 (D9)
- net BIN2: now also U1.14 (IN_B2)
- net STBY: now reaches A1.7 (D4)
- net STBY: now also U1.12 (STNDBY)
- net AIN1: now reaches U1.10 (IN_A2)
- net AIN1: now also A1.9 (D6)
- net AIN2: now reaches U1.11 (IN_A1)
- net BIN1: now reaches U1.13 (IN_B1)
Other:
- note added: "Device refernece :"
- moved on the sheet: A1

Commit message: well theres a second version now
Parts:
- removed C1: C, Capacitor_THT:C_Disc_D5.0mm_W2.5mm_P2.50mm, symbol Device:C
- added SW3: SW_SPST, Button_Switch_THT:SW_CuK_OS102011MA1QN1_SPDT_Angled, symbol Switch:SW_SPST
- J2, J3: footprint TerminalBlock:TerminalBlock_Altech_AK300-2_P5.00mm -> sche:MOTORmount
Connections:
- net VS: now also SW3.1 (A); no longer U2.1 (VI)
- new net: SW3.2 (B), U2.1 (VI)
Changed lines of the file:
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@@
   (junction (at 218.44 149.86) (diameter 0) (color 0 0 0 0)
   )
-  (junction (at 210.82 39.37) (diameter 0) (color 0 0 0 0)
-  )
   (junction (at 27.94 132.08) (diameter 0) (color 0 0 0 0)
   )
@@
     (stroke (width 0) (type default))
   )
-  (wire (pts (xy 210.82 49.53) (xy 224.79 49.53))
-    (stroke (width 0) (type default))
-  )
   (wire (pts (xy 219.71 102.87) (xy 219.71 104.14))
     (stroke (width 0) (type default))
@@
     (stroke (width 0) (type default))
   )
+  (wire (pts (xy 200.66 35.56) (xy 200.66 39.37))
+    (stroke (width 0) (type default))
+  )
   (wire (pts (xy 97.79 58.42) (xy 104.14 58.42))
     (stroke (width 0) (type default))
@@
     (stroke (width 0) (type default))
   )
-  (wire (pts (xy 210.82 39.37) (xy 210.82 40.64))
-    (stroke (width 0) (type default))
-  )
   (wire (pts (xy 69.85 144.78) (xy 77.47 144.78))
     (stroke (width 0) (type default))
@@
     (stroke (width 0) (type default))
   )
+  (wire (pts (xy 214.63 39.37) (xy 217.17 39.37))
+    (stroke (width 0) (type default))
+  )
   (wire (pts (xy 97.79 60.96) (xy 104.14 60.96))
     (stroke (width 0) (type default))
@@
     (stroke (width 0) (type default))
   )
-  (wire (pts (xy 210.82 35.56) (xy 210.82 39.37))
-    (stroke (width 0) (type default))
-  )
   (wire (pts (xy 121.92 158.75) (xy 115.57 158.75))
     (stroke (width 0) (type default))
@@
     (stroke (width 0) (type default))
   )
-  (wire (pts (xy 210.82 48.26) (xy 210.82 49.53))
-    (stroke (width 0) (type default))
-  )
   (wire (pts (xy 64.77 55.88) (xy 72.39 55.88))
     (stroke (width 0) (type default))
@@
     (stroke (width 0) (type default))
   )
-  (wire (pts (xy 210.82 39.37) (xy 217.17 39.37))
-    (stroke (width 0) (type default))
-  )
   (wire (pts (xy 215.9 149.86) (xy 218.44 149.86))
     (stroke (width 0) (type default))
@@
     (stroke (width 0) (type default))
   )
+  (wire (pts (xy 200.66 39.37) (xy 204.47 39.37))
+    (stroke (width 0) (type default))
+  )
   (wire (pts (xy 85.09 83.82) (xy 85.09 86.36))
     (stroke (width 0) (type default))
@@
       (effects (font (size 1.27 1.27)) (justify left))
     )
-    (property "Footprint" "TerminalBlock:TerminalBlock_Altech_AK300-2_P5.00mm" (at 82.55 129.54 0)
+    (property "Footprint" "sche:MOTORmount" (at 82.55 129.54 0)
       (effects (font (size 1.27 1.27)) hide)
     )
@@
     )
   )
-  (symbol (lib_id "power:VS") (at 210.82 35.56 0) (unit 1)
+  (symbol (lib_id "power:VS") (at 200.66 35.56 0) (unit 1)
     (in_bom yes) (on_board yes) (dnp no) (fields_autoplaced)
-    (property "Reference" "#PWR010" (at 205.74 39.37 0)
+    (property "Reference" "#PWR010" (at 195.58 39.37 0)
       (effects (font (size 1.27 1.27)) hide)
     )
-    (property "Value" "VS" (at 210.82 31.75 0)
+    (property "Value" "VS" (at 200.66 31.75 0)
       (effects (font (size 1.27 1.27)))
     )
-    (property "Footprint" "" (at 210.82 35.56 0)
+    (property "Footprint" "" (at 200.66 35.56 0)
       (effects (font (size 1.27 1.27)) hide)
     )
-    (property "Datasheet" "" (at 210.82 35.56 0)
+    (property "Datasheet" "" (at 200.66 35.56 0)
       (effects (font (size 1.27 1.27)) hide)
     )
@@
     )
   )
-  (symbol (lib_id "Device:C") (at 210.82 44.45 0) (unit 1)
+  (symbol (lib_id "Switch:SW_SPST") (at 209.55 39.37 0) (unit 1)
     (in_bom yes) (on_board yes) (dnp no) (fields_autoplaced)
-    (property "Reference" "C1" (at 214.63 43.815 0)
-      (effects (font (size 1.27 1.27)) (justify left))
+    (property "Reference" "SW3" (at 209.55 34.29 0)
+      (effects (font (size 1.27 1.27)))
     )
-    (property "Value" "C" (at 214.63 46.355 0)
-      (effects (font (size 1.27 1.27)) (justify left))
+    (property "Value" "SW_SPST" (at 209.55 36.83 0)
+      (effects (font (size 1.27 1.27)))
     )
-    (property "Footprint" "Capacitor_THT:C_Disc_D5.0mm_W2.5mm_P2.50mm" (at 211.7852 48.26 0)
+    (property "Footprint" "Button_Switch_THT:SW_CuK_OS102011MA1QN1_SPDT_Angled" (at 209.55 39.37 0)
       (effects (font (size 1.27 1.27)) hide)
     )
-    (property "Datasheet" "~" (at 210.82 44.45 0)
+    (property "Datasheet" "~" (at 209.55 39.37 0)
       (effects (font (size 1.27 1.27)) hide)
     )
@@
       (project "fastlinefollower_tbfng"
         (path "/0073a757-8926-4bfa-90ed-7735299474ab"
-          (reference "C1") (unit 1)
-        )
-      )
-      (project "fastlinefollower"
-        (path "/12d22a33-b5ed-48ef-8dcf-cecf4d5020b2"
-          (reference "C1") (unit 1)
+          (reference "SW3") (unit 1)
         )
       )
@@
       (effects (font (size 1.27 1.27)) (justify left))
     )
-    (property "Footprint" "TerminalBlock:TerminalBlock_Altech_AK300-2_P5.00mm" (at 82.55 142.24 0)
+    (property "Footprint" "sche:MOTORmount" (at 82.55 142.24 0)
       (effects (font (size 1.27 1.27)) hide)
     )
