File: fastlinefollower_tbfng_v1.kicad_pcb (KiCad board)
At the start: 2 copper layers, 100 x 70 mm, 10 parts, among them J1 IR_conn, J2 Motor1, J3 Motor2, SW1 Run, SW2 Calibrate, U1 TB6612FNG_Module, U2 LM7805_TO220

Commit message: well theres a second version now
Parts:
- removed C1: C, Capacitor_THT:C_Disc_D5.0mm_W2.5mm_P2.50mm
- added SW3: SW_SPST, Button_Switch_THT:SW_CuK_OS102011MA1QN1_SPDT_Angled, F.Cu at (108.0, 123.1)
- J2, J3: footprint TerminalBlock:TerminalBlock_Altech_AK300-2_P5.00mm -> sche:MOTORmount
- moved J2 16.3 mm to (123.0, 142.0)
- moved J3 13.8 mm to (159.1, 142.0)
- moved U2 11.1 mm to (109.0, 112.0)
- moved C2 9.83 mm to (114.0, 107.0)
- moved SW1 9.10 mm to (175.2, 110.5)
- moved SW2 9.10 mm to (168.8, 118.8)
Connections:
- U2 pad 1: VS -> Net-(SW3-B)
Routing:
- net +5V: track 222.1 -> 117.7 mm
- net VS: track 70.7 -> 0.33 mm
- net Net-(SW3-B): track 0.00 -> 13.7 mm
- net /M2_B: track 27.0 -> 15.2 mm
- net /M1_A: track 31.8 -> 20.1 mm
- net /M2_A: track 32.4 -> 23.3 mm
- net /M1_B: track 37.8 -> 28.8 mm
- net /RUN: track 49.5 -> 41.1 mm
- net /CAL: track 56.6 -> 50.8 mm
Other:
- board size 100 x 70 mm -> 90 x 65 mm
- board text added: "Battery"
- board text added: "Motor 1"
- board text added: "Motor 2"

Commit message: new layout
Parts:
- added C1: C, Capacitor_THT:C_Disc_D3.4mm_W2.1mm_P2.50mm, F.Cu at (129.0, 146.5)
- added C3: C, Capacitor_THT:C_Disc_D3.4mm_W2.1mm_P2.50mm, F.Cu at (153.0, 143.5)
- SW1, SW2: footprint Button_Switch_THT:SW_PUSH_6mm -> sche:SPST_Pushbutton
- SW3: footprint Button_Switch_THT:SW_CuK_OS102011MA1QN1_SPDT_Angled -> sche:SPDT_Slidebutton
- moved SW3 11.9 mm to (110.5, 111.5), turned to 0 degrees
- moved SW1 9.50 mm to (171.0, 102.0)
- moved SW2 9.03 mm to (171.0, 110.0), turned to 180 degrees
- moved C2 6.08 mm to (113.0, 101.0), turned to 90 degrees
- moved U2 5.11 mm to (108.0, 107.0), turned to 0 degrees
Connections:
- SW1 pad 1: +5V -> /RUN
- SW1 pad 2: /RUN -> GND
- SW2 pad 1: +5V -> /CAL
- SW2 pad 2: /CAL -> GND
- SW3 pad 1: VS -> GND
- SW3 pad 2: Net-(SW3-B) -> /Vin
- SW3 pad 3: (no net) -> VS
- U1 pad 1: VS -> /Vin
- U2 pad 1: Net-(SW3-B) -> /Vin
Routing:
- net /Vin: track 0.00 -> 81.1 mm
- net +5V: track 117.7 -> 160.3 mm
- net Net-(SW3-B): track 13.7 -> 0.00 mm
- net /CAL: track 50.8 -> 38.0 mm
- net /RUN: track 41.1 -> 43.3 mm
- net /M2_A: track 23.3 -> 24.5 mm
- net /M2_B: track 15.2 -> 16.2 mm
Other:
- outline, holes or cut-outs redrawn
