File: fastlinefollower_tbfng_v2.kicad_pcb (KiCad board)
At the start: 2 copper layers, 90 x 70 mm, 12 parts, among them J1 IR_conn, J2 Motor1, J3 Motor2, SW1 Run, SW2 Calibrate, SW3 SW_SPST, U1 TB6612FNG_Module, U2 LM7805_TO220

Commit message: final twicks
Parts:
- added J4: POWER, TerminalBlock:TerminalBlock_bornier-2_P5.08mm, F.Cu at (110.5, 78.0)
- added REF**: draiclogo_small, sche:draiclogo_small, F.Cu at (114.0, 112.0)
- moved SW3 65.4 mm to (50.5, 86.0), turned to 180 degrees
- moved A1 65.3 mm to (61.0, 105.1)
- moved C2 65.3 mm to (51.5, 97.5)
- moved J1 65.3 mm to (91.4, 84.5)
- moved J2 65.3 mm to (62.0, 118.5)
- moved C1 65.3 mm to (68.0, 123.0)
- moved C3 65.3 mm to (92.0, 120.0)
- moved J3 65.3 mm to (98.1, 118.5)
- moved SW1 65.3 mm to (110.0, 90.0)
- moved SW2 65.3 mm to (110.0, 97.5)
- moved U2 65.3 mm to (48.0, 92.9)
- moved U1 65.3 mm to (88.9, 130.3)
Routing:
- net VS: track 0.00 -> 60.7 mm
- net /M2_A: track 24.7 -> 23.6 mm
- net /Vin: track 62.1 -> 62.9 mm
Other:
- outline, holes or cut-outs redrawn
