File: fastlinefollower_tbfng_v2.kicad_sch (KiCad schematic)
At the start: 12 parts, among them J1 IR_conn, J2 Motor1, J3 Motor2, SW1 Run, SW2 Calibrate, SW3 SW_SPST, U1 TB6612FNG_Module, U2 LM7805_TO220

Commit message: new layout
Connections:
- net +5V: now also J1.9 (Pin_9); no longer J1.1 (Pin_1)
- net IR1: now also J1.1 (Pin_1); no longer J1.2 (Pin_2)
- net IR2: now also J1.2 (Pin_2); no longer J1.3 (Pin_3)
- net IR3: now also J1.3 (Pin_3); no longer J1.4 (Pin_4)
- net IR4: now also J1.4 (Pin_4); no longer J1.5 (Pin_5)
- net IR5: now also J1.5 (Pin_5); no longer J1.6 (Pin_6)
- net IR6: now also J1.6 (Pin_6); no longer J1.7 (Pin_7)
- net IR7: now also J1.7 (Pin_7); no longer J1.8 (Pin_8)
- net IR8: now also J1.8 (Pin_8); no longer J1.9 (Pin_9)
Changed lines of the file:
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@@
     (stroke (width 0) (type default))
   )
-  (wire (pts (xy 119.38 148.59) (xy 121.92 148.59))
+  (wire (pts (xy 111.76 168.91) (xy 121.92 168.91))
     (stroke (width 0) (type default))
   )
@@
     (stroke (width 0) (type default))
   )
-  (wire (pts (xy 121.92 166.37) (xy 115.57 166.37))
+  (wire (pts (xy 121.92 163.83) (xy 115.57 163.83))
     (stroke (width 0) (type default))
   )
@@
     (stroke (width 0) (type default))
   )
-  (wire (pts (xy 121.92 163.83) (xy 115.57 163.83))
+  (wire (pts (xy 121.92 161.29) (xy 115.57 161.29))
     (stroke (width 0) (type default))
   )
@@
     (stroke (width 0) (type default))
   )
-  (wire (pts (xy 121.92 158.75) (xy 115.57 158.75))
+  (wire (pts (xy 121.92 156.21) (xy 115.57 156.21))
     (stroke (width 0) (type default))
   )
-  (wire (pts (xy 121.92 156.21) (xy 115.57 156.21))
+  (wire (pts (xy 121.92 153.67) (xy 115.57 153.67))
     (stroke (width 0) (type default))
   )
@@
     (stroke (width 0) (type default))
   )
-  (wire (pts (xy 121.92 153.67) (xy 115.57 153.67))
+  (wire (pts (xy 121.92 151.13) (xy 115.57 151.13))
     (stroke (width 0) (type default))
   )
@@
     (stroke (width 0) (type default))
   )
-  (wire (pts (xy 119.38 146.05) (xy 119.38 148.59))
+  (wire (pts (xy 111.76 166.37) (xy 111.76 168.91))
     (stroke (width 0) (type default))
   )
@@
     (stroke (width 0) (type default))
   )
-  (wire (pts (xy 121.92 161.29) (xy 115.57 161.29))
+  (wire (pts (xy 121.92 158.75) (xy 115.57 158.75))
     (stroke (width 0) (type default))
   )
@@
     (stroke (width 0) (type default))
   )
-  (wire (pts (xy 121.92 151.13) (xy 115.57 151.13))
+  (wire (pts (xy 121.92 148.59) (xy 115.57 148.59))
     (stroke (width 0) (type default))
   )
-  (wire (pts (xy 121.92 168.91) (xy 115.57 168.91))
+  (wire (pts (xy 121.92 166.37) (xy 115.57 166.37))
     (stroke (width 0) (type default))
   )
@@
     (effects (font (size 1.27 1.27)) (justify left bottom))
   )
-  (label "IR1" (at 115.57 151.13 0) (fields_autoplaced)
+  (label "IR1" (at 115.57 148.59 0) (fields_autoplaced)
     (effects (font (size 1.27 1.27)) (justify left bottom))
   )
@@
     (effects (font (size 1.27 1.27)) (justify left bottom))
   )
-  (label "IR2" (at 115.57 153.67 0) (fields_autoplaced)
+  (label "IR2" (at 115.57 151.13 0) (fields_autoplaced)
     (effects (font (size 1.27 1.27)) (justify left bottom))
   )
@@
     (effects (font (size 1.27 1.27)) (justify right bottom))
   )
-  (label "IR4" (at 115.57 158.75 0) (fields_autoplaced)
+  (label "IR4" (at 115.57 156.21 0) (fields_autoplaced)
     (effects (font (size 1.27 1.27)) (justify left bottom))
   )
@@
     (effects (font (size 1.27 1.27)) (justify right bottom))
   )
-  (label "IR5" (at 115.57 161.29 0) (fields_autoplaced)
+  (label "IR5" (at 115.57 158.75 0) (fields_autoplaced)
     (effects (font (size 1.27 1.27)) (justify left bottom))
   )
@@
     (effects (font (size 1.27 1.27)) (justify left bottom))
   )
-  (label "IR3" (at 115.57 156.21 0) (fields_autoplaced)
+  (label "IR3" (at 115.57 153.67 0) (fields_autoplaced)
     (effects (font (size 1.27 1.27)) (justify left bottom))
   )
@@
     (effects (font (size 1.27 1.27)) (justify left bottom))
   )
-  (label "IR6" (at 115.57 163.83 0) (fields_autoplaced)
+  (label "IR6" (at 115.57 161.29 0) (fields_autoplaced)
     (effects (font (size 1.27 1.27)) (justify left bottom))
   )
@@
     (effects (font (size 1.27 1.27)) (justify left bottom))
   )
-  (label "IR7" (at 115.57 166.37 0) (fields_autoplaced)
+  (label "IR7" (at 115.57 163.83 0) (fields_autoplaced)
     (effects (font (size 1.27 1.27)) (justify left bottom))
   )
@@
     (effects (font (size 1.27 1.27)) (justify left bottom))
   )
-  (label "IR8" (at 115.57 168.91 0) (fields_autoplaced)
+  (label "IR8" (at 115.57 166.37 0) (fields_autoplaced)
     (effects (font (size 1.27 1.27)) (justify left bottom))
   )
@@
     (pin "9")
     (instances
-      (project "fastlinefollower_tbfng"
+      (project "fastlinefollower_tbfng_v2"
         (path "/0073a757-8926-4bfa-90ed-7735299474ab"
           (reference "A1") (unit 1)
@@
     (pin "1")
     (instances
-      (project "fastlinefollower_tbfng"
+      (project "fastlinefollower_tbfng_v2"
         (path "/0073a757-8926-4bfa-90ed-7735299474ab"
           (reference "#PWR02") (unit 1)
@@
     (pin "2")
     (instances
-      (project "fastlinefollower_tbfng"
+      (project "fastlinefollower_tbfng_v2"
         (path "/0073a757-8926-4bfa-90ed-7735299474ab"
           (reference "C1") (unit 1)
@@
     (pin "3")
     (instances
-      (project "fastlinefollower_tbfng"
+      (project "fastlinefollower_tbfng_v2"
         (path "/0073a757-8926-4bfa-90ed-7735299474ab"
           (reference "U2") (unit 1)
@@
     (pin "9")
     (instances
-      (project "fastlinefollower_tbfng"
+      (project "fastlinefollower_tbfng_v2"
         (path "/0073a757-8926-4bfa-90ed-7735299474ab"
           (reference "U1") (unit 1)
@@
     (pin "2")
     (instances
-      (project "fastlinefollower_tbfng"
+      (project "fastlinefollower_tbfng_v2"
         (path "/0073a757-8926-4bfa-90ed-7735299474ab"
           (reference "J2") (unit 1)
@@
     (pin "2")
     (instances
-      (project "fastlinefollower_tbfng"
+      (project "fastlinefollower_tbfng_v2"
         (path "/0073a757-8926-4bfa-90ed-7735299474ab"
           (reference "SW1") (unit 1)
@@
     (pin "2")
     (instances
-      (project "fastlinefollower_tbfng"
+      (project "fastlinefollower_tbfng_v2"
         (path "/0073a757-8926-4bfa-90ed-7735299474ab"
           (reference "SW2") (unit 1)
@@
     (pin "1")
     (instances
-      (project "fastlinefollower_tbfng"
+      (project "fastlinefollower_tbfng_v2"
         (path "/0073a757-8926-4bfa-90ed-7735299474ab"
           (reference "#PWR010") (unit 1)
@@
     (pin "1")
     (instances
-      (project "fastlinefollower_tbfng"
+      (project "fastlinefollower_tbfng_v2"
         (path "/0073a757-8926-4bfa-90ed-7735299474ab"
           (reference "#PWR08") (unit 1)
@@
     (pin "2")
     (instances
-      (project "fastlinefollower_tbfng"
+      (project "fastlinefollower_tbfng_v2"
         (path "/0073a757-8926-4bfa-90ed-7735299474ab"
           (reference "C3") (unit 1)
@@
     )
   )
-  (symbol (lib_id "power:+5V") (at 119.38 146.05 0) (unit 1)
+  (symbol (lib_id "power:+5V") (at 111.76 166.37 0) (unit 1)
     (in_bom yes) (on_board yes) (dnp no) (fields_autoplaced)
-    (property "Reference" "#PWR015" (at 119.38 149.86 0)
+    (property "Reference" "#PWR015" (at 111.76 170.18 0)
       (effects (font (size 1.27 1.27)) hide)
     )
-    (property "Value" "+5V" (at 119.38 142.24 0)
+    (property "Value" "+5V" (at 111.76 162.56 0)
       (effects (font (size 1.27 1.27)))
     )
-    (property "Footprint" "" (at 119.38 146.05 0)
+    (property "Footprint" "" (at 111.76 166.37 0)
       (effects (font (size 1.27 1.27)) hide)
     )
-    (property "Datasheet" "" (at 119.38 146.05 0)
+    (property "Datasheet" "" (at 111.76 166.37 0)
       (effects (font (size 1.27 1.27)) hide)
     )
     (pin "1")
     (instances
-      (project "fastlinefollower_tbfng"
+      (project "fastlinefollower_tbfng_v2"
         (path "/0073a757-8926-4bfa-90ed-7735299474ab"
           (reference "#PWR015") (unit 1)
@@
     (pin "1")
     (instances
-      (project "fastlinefollower_tbfng"
+      (project "fastlinefollower_tbfng_v2"
         (path "/0073a757-8926-4bfa-90ed-7735299474ab"
           (reference "#PWR07") (unit 1)
@@
     (pin "1")
     (instances
-      (project "fastlinefollower_tbfng"
+      (project "fastlinefollower_tbfng_v2"
         (path "/0073a757-8926-4bfa-90ed-7735299474ab"
           (reference "#PWR01") (unit 1)
@@
     (pin "1")
     (instances
-      (project "fastlinefollower_tbfng"
+      (project "fastlinefollower_tbfng_v2"
         (path "/0073a757-8926-4bfa-90ed-7735299474ab"
           (reference "#PWR06") (unit 1)
@@
     (pin "3")
     (instances
-      (project "fastlinefollower_tbfng"
+      (project "fastlinefollower_tbfng_v2"
         (path "/0073a757-8926-4bfa-90ed-7735299474ab"
           (reference "SW3") (unit 1)
@@
     (pin "2")
     (instances
-      (project "fastlinefollower_tbfng"
+      (project "fastlinefollower_tbfng_v2"
         (path "/0073a757-8926-4bfa-90ed-7735299474ab"
           (reference "C2") (unit 1)
@@
     (pin "9")
     (instances
-      (project "fastlinefollower_tbfng"
+      (project "fastlinefollower_tbfng_v2"
         (path "/0073a757-8926-4bfa-90ed-7735299474ab"
           (reference "J1") (unit 1)
@@
     (pin "2")
     (instances
-      (project "fastlinefollower_tbfng"
+      (project "fastlinefollower_tbfng_v2"
         (path "/0073a757-8926-4bfa-90ed-7735299474ab"
           (reference "J3") (unit 1)
@@
     (pin "1")
     (instances
-      (project "fastlinefollower_tbfng"
+      (project "fastlinefollower_tbfng_v2"
         (path "/0073a757-8926-4bfa-90ed-7735299474ab"
           (reference "#PWR05") (unit 1)
@@
     (pin "1")
     (instances
-      (project "fastlinefollower_tbfng"
+      (project "fastlinefollower_tbfng_v2"
         (path "/0073a757-8926-4bfa-90ed-7735299474ab"
           (reference "#PWR016") (unit 1)
@@
     (pin "1")
     (instances
-      (project "fastlinefollower_tbfng"
+      (project "fastlinefollower_tbfng_v2"
         (path "/0073a757-8926-4bfa-90ed-7735299474ab"
           (reference "#PWR04") (unit 1)
@@
     (pin "1")
     (instances
-      (project "fastlinefollower_tbfng"
+      (project "fastlinefollower_tbfng_v2"
         (path "/0073a757-8926-4bfa-90ed-7735299474ab"
           (reference "#PWR03") (unit 1)

Commit message: final twicks
Parts:
- added J4: POWER, TerminalBlock:TerminalBlock_bornier-2_P5.08mm, symbol Connector:Screw_Terminal_01x02
Connections:
- net GND: now also J4.1 (Pin_1)
- net VS: now also J4.2 (Pin_2)
Other:
- note added: "Arduino Nano"
- note added: "Fastest Line Follower"
- note added: "Inputs"
- note added: "Motor Driver and Output"
- note added: "Power Supply"
- note added: "This a basic line follower that is using an array of 8 IR's to follow a line. uC reads analog values from IR array and using PID and Polulu's Line follower library will follow a line."
- company: (none) -> DRAIC
- title: (none) -> Fastest Line Follower
- moved on the sheet: A1, C1, C2, C3, J1, J2, J3, SW1, SW2, SW3, U1, U2
